Commit message: franka_description_custom/** -> ros_objslampp_panda

File: ros/ros_objslampp_panda/robots/panda_arm_suction_gripper.urdf.xacro (robot description, xacro)
@@ -169,16 +169,6 @@
     </joint>
   </xacro:macro>
-  <xacro:include filename="$(find franka_description_custom)/robots/suction/suction_gripper.xacro"/>
-  <xacro:include filename="$(find franka_description_custom)/robots/scene/table.xacro"/>
-  <xacro:include filename="$(find franka_description_custom)/robots/scene/left_wall.xacro"/>
-  <xacro:include filename="$(find franka_description_custom)/robots/scene/front_wall.xacro"/>
-  <xacro:include filename="$(find franka_description_custom)/robots/scene/target_box.xacro"/>
-  <xacro:include filename="$(find franka_description_custom)/robots/scene/distractor_box.xacro"/>
+  <xacro:include filename="$(find ros_objslampp_panda)/robots/suction/suction_gripper.xacro"/>
   <xacro:panda_arm />
   <xacro:suction_gripper ns="panda" rpy="${pi} 0 ${-pi/4}" xyz="0 0 0.0065" connected_to="panda_link8"/>
-  <xacro:table ns="panda" rpy="0 0 0" xyz="0.68 0 0.0375" connected_to="panda_link0"/>
-  <xacro:left_wall ns="panda" rpy="${pi/2} 0 0" xyz="0.68 0.65 0.6" connected_to="panda_link0"/>
-  <xacro:front_wall ns="panda" rpy="0 ${pi/2} 0" xyz="1.33 0 0.6" connected_to="panda_link0"/>
-  <xacro:target_box ns="panda" rpy="0 0 0" xyz="0.6 -0.45 0.075" connected_to="panda_link0"/>
-  <xacro:distractor_box ns="panda" rpy="0 0 0" xyz="0.665 0.445 0.0775" connected_to="panda_link0"/>
 </robot>

File: ros/ros_objslampp_panda/robots/panda_arm_suction_gripper_and_scene.urdf.xacro (robot description, xacro)
@@ -169,8 +169,8 @@
     </joint>
   </xacro:macro>
-  <xacro:include filename="$(find franka_description_custom)/robots/suction/suction_gripper.xacro"/>
-  <xacro:include filename="$(find franka_description_custom)/robots/scene/table.xacro"/>
-  <xacro:include filename="$(find franka_description_custom)/robots/scene/left_wall.xacro"/>
-  <xacro:include filename="$(find franka_description_custom)/robots/scene/front_wall.xacro"/>
+  <xacro:include filename="$(find ros_objslampp_panda)/robots/suction/suction_gripper.xacro"/>
+  <xacro:include filename="$(find ros_objslampp_panda)/robots/scene/table.xacro"/>
+  <xacro:include filename="$(find ros_objslampp_panda)/robots/scene/left_wall.xacro"/>
+  <xacro:include filename="$(find ros_objslampp_panda)/robots/scene/front_wall.xacro"/>
   <xacro:panda_arm />
   <xacro:suction_gripper ns="panda" rpy="${pi} 0 ${-pi/4}" xyz="0 0 0.0065" connected_to="panda_link8"/>

File: ros/ros_objslampp_panda/robots/panda_arm_suction_gripper_objslampp.urdf.xacro (robot description, xacro)
@@ -169,6 +169,16 @@
     </joint>
   </xacro:macro>
-  <xacro:include filename="$(find franka_description_custom)/robots/suction/suction_gripper.xacro"/>
+  <xacro:include filename="$(find ros_objslampp_panda)/robots/suction/suction_gripper.xacro"/>
+  <xacro:include filename="$(find ros_objslampp_panda)/robots/scene/table.xacro"/>
+  <xacro:include filename="$(find ros_objslampp_panda)/robots/scene/left_wall.xacro"/>
+  <xacro:include filename="$(find ros_objslampp_panda)/robots/scene/front_wall.xacro"/>
+  <xacro:include filename="$(find ros_objslampp_panda)/robots/scene/target_box.xacro"/>
+  <xacro:include filename="$(find ros_objslampp_panda)/robots/scene/distractor_box.xacro"/>
   <xacro:panda_arm />
   <xacro:suction_gripper ns="panda" rpy="${pi} 0 ${-pi/4}" xyz="0 0 0.0065" connected_to="panda_link8"/>
+  <xacro:table ns="panda" rpy="0 0 0" xyz="0.68 0 0.0375" connected_to="panda_link0"/>
+  <xacro:left_wall ns="panda" rpy="${pi/2} 0 0" xyz="0.68 0.65 0.6" connected_to="panda_link0"/>
+  <xacro:front_wall ns="panda" rpy="0 ${pi/2} 0" xyz="1.33 0 0.6" connected_to="panda_link0"/>
+  <xacro:target_box ns="panda" rpy="0 0 0" xyz="0.6 -0.45 0.075" connected_to="panda_link0"/>
+  <xacro:distractor_box ns="panda" rpy="0 0 0" xyz="0.665 0.445 0.0775" connected_to="panda_link0"/>
 </robot>

File: ros/ros_objslampp_panda/robots/suction/suction_gripper.xacro (robot description, xacro)
@@ -18,5 +18,5 @@
       <visual>
         <geometry>
-          <mesh filename="package://franka_description_custom/meshes/visual/suction_mount.stl"/>
+          <mesh filename="package://ros_objslampp_panda/meshes/visual/suction_mount.stl"/>
         </geometry>
         <material name="black"/>
@@ -32,5 +32,5 @@
       <visual>
         <geometry>
-          <mesh filename="package://franka_description_custom/meshes/visual/suction_cup.stl"/>
+          <mesh filename="package://ros_objslampp_panda/meshes/visual/suction_cup.stl"/>
         </geometry>
         <material name="green"/>

Commit message: Simplify panda_arm_suction_gripper.urdf.xacro

File: ros/ros_objslampp_panda/robots/panda_arm_suction_gripper.urdf.xacro (robot description, xacro)
@@ -1,174 +1,7 @@
 <?xml version="1.0" encoding="utf-8"?>
 <robot xmlns:xacro="http://www.ros.org/wiki/xacro" name="panda">
-  <xacro:macro name="panda_arm" params="arm_id:='panda' description_pkg:='franka_description' connected_to:='' xyz:='0 0 0' rpy:='0 0 0'">
-    <xacro:unless value="${not connected_to}">
-      <joint name="${arm_id}_joint_${connected_to}" type="fixed">
-        <parent link="${connected_to}"/>
-        <child link="${arm_id}_link0"/>
-        <origin rpy="${rpy}" xyz="${xyz}"/>
-      </joint>
-    </xacro:unless>
-    <link name="${arm_id}_link0">
-      <visual>
-        <geometry>
-          <mesh filename="package://${description_pkg}/meshes/visual/link0.dae"/>
-        </geometry>
-      </visual>
-      <collision>
-        <geometry>
-          <mesh filename="package://${description_pkg}/meshes/collision/link0.stl"/>
-        </geometry>
-      </collision>
-    </link>
-    <link name="${arm_id}_link1">
-      <visual>
-        <geometry>
-          <mesh filename="package://${description_pkg}/meshes/visual/link1.dae"/>
-        </geometry>
-      </visual>
-      <collision>
-        <geometry>
-          <mesh filename="package://${description_pkg}/meshes/collision/link1.stl"/>
-        </geometry>
-      </collision>
-    </link>
-    <joint name="${arm_id}_joint1" type="revolute">
-      <safety_controller k_position="100.0" k_velocity="40.0" soft_lower_limit="-2.8973" soft_upper_limit="2.8973"/>
-      <origin rpy="0 0 0" xyz="0 0 0.333"/>
-      <parent link="${arm_id}_link0"/>
-      <child link="${arm_id}_link1"/>
-      <axis xyz="0 0 1"/>
-      <limit effort="87" lower="-2.8" upper="2.8" velocity="2.1750"/>
-    </joint>
-    <link name="${arm_id}_link2">
-      <visual>
-        <geometry>
-          <mesh filename="package://${description_pkg}/meshes/visual/link2.dae"/>
-        </geometry>
-      </visual>
-      <collision>
-        <geometry>
-          <mesh filename="package://${description_pkg}/meshes/collision/link2.stl"/>
-        </geometry>
-      </collision>
-    </link>
-    <joint name="${arm_id}_joint2" type="revolute">
-      <safety_controller k_position="100.0" k_velocity="40.0" soft_lower_limit="-1.7628" soft_upper_limit="1.7628"/>
-      <origin rpy="${-pi/2} 0 0" xyz="0 0 0"/>
-      <parent link="${arm_id}_link1"/>
-      <child link="${arm_id}_link2"/>
-      <axis xyz="0 0 1"/>
-      <limit effort="87" lower="-1.7" upper="1.7" velocity="2.1750"/>
-    </joint>
-    <link name="${arm_id}_link3">
-      <visual>
-        <geometry>
-          <mesh filename="package://${description_pkg}/meshes/visual/link3.dae"/>
-        </geometry>
-      </visual>
-      <collision>
-        <geometry>
-          <mesh filename="package://${description_pkg}/meshes/collision/link3.stl"/>
-        </geometry>
-      </collision>
-    </link>
-    <joint name="${arm_id}_joint3" type="revolute">
-      <safety_controller k_position="100.0" k_velocity="40.0" soft_lower_limit="-2.8973" soft_upper_limit="2.8973"/>
-      <origin rpy="${pi/2} 0 0" xyz="0 -0.316 0"/>
-      <parent link="${arm_id}_link2"/>
-      <child link="${arm_id}_link3"/>
-      <axis xyz="0 0 1"/>
-      <limit effort="87" lower="-2.8" upper="2.8" velocity="2.1750"/>
-    </joint>
-    <link name="${arm_id}_link4">
-      <visual>
-        <geometry>
-          <mesh filename="package://${description_pkg}/meshes/visual/link4.dae"/>
-        </geometry>
-      </visual>
-      <collision>
-        <geometry>
-          <mesh filename="package://${description_pkg}/meshes/collision/link4.stl"/>
-        </geometry>
-      </collision>
-    </link>
-    <joint name="${arm_id}_joint4" type="revolute">
-      <safety_controller k_position="100.0" k_velocity="40.0" soft_lower_limit="-3.0718" soft_upper_limit="-0.0698"/>
-      <origin rpy="${pi/2} 0 0" xyz="0.0825 0 0"/>
-      <parent link="${arm_id}_link3"/>
-      <child link="${arm_id}_link4"/>
-      <axis xyz="0 0 1"/>
-      <limit effort="87" lower="-3.0" upper="0.0" velocity="2.1750"/>
-    </joint>
-    <link name="${arm_id}_link5">
-      <visual>
-        <geometry>
-          <mesh filename="package://${description_pkg}/meshes/visual/link5.dae"/>
-        </geometry>
-      </visual>
-      <collision>
-        <geometry>
-          <mesh filename="package://${description_pkg}/meshes/collision/link5.stl"/>
-        </geometry>
-      </collision>
-    </link>
-    <joint name="${arm_id}_joint5" type="revolute">
-      <safety_controller k_position="100.0" k_velocity="40.0" soft_lower_limit="-2.8973" soft_upper_limit="2.8973"/>
-      <origin rpy="${-pi/2} 0 0" xyz="-0.0825 0.384 0"/>
-      <parent link="${arm_id}_link4"/>
-      <child link="${arm_id}_link5"/>
-      <axis xyz="0 0 1"/>
-      <limit effort="12" lower="-2.8" upper="2.8" velocity="2.6100"/>
-    </joint>
-    <link name="${arm_id}_link6">
-      <visual>
-        <geometry>
-          <mesh filename="package://${description_pkg}/meshes/visual/link6.dae"/>
-        </geometry>
-      </visual>
-      <collision>
-        <geometry>
-          <mesh filename="package://${description_pkg}/meshes/collision/link6.stl"/>
-        </geometry>
-      </collision>
-    </link>
-    <joint name="${arm_id}_joint6" type="revolute">
-      <safety_controller k_position="100.0" k_velocity="40.0" soft_lower_limit="-0.0175" soft_upper_limit="3.7525"/>
-      <origin rpy="${pi/2} 0 0" xyz="0 0 0"/>
-      <parent link="${arm_id}_link5"/>
-      <child link="${arm_id}_link6"/>
-      <axis xyz="0 0 1"/>
-      <limit effort="12" lower="0.0" upper="3.7" velocity="2.6100"/>
-    </joint>
-    <link name="${arm_id}_link7">
-      <visual>
-        <geometry>
-          <mesh filename="package://${description_pkg}/meshes/visual/link7.dae"/>
-        </geometry>
-      </visual>
-      <collision>
-        <geometry>
-          <mesh filename="package://${description_pkg}/meshes/collision/link7.stl"/>
-        </geometry>
-      </collision>
-    </link>
-    <joint name="${arm_id}_joint7" type="revolute">
-      <safety_controller k_position="100.0" k_velocity="40.0" soft_lower_limit="-2.8973" soft_upper_limit="2.8973"/>
-      <origin rpy="${pi/2} 0 0" xyz="0.088 0 0"/>
-      <parent link="${arm_id}_link6"/>
-      <child link="${arm_id}_link7"/>
-      <axis xyz="0 0 1"/>
-      <limit effort="12" lower="${-pi/4}" upper="${3*pi/4}" velocity="2.6100"/>
-    </joint>
-    <link name="${arm_id}_link8"/>
-    <joint name="${arm_id}_joint8" type="fixed">
-      <origin rpy="0 0 0" xyz="0 0 0.107"/>
-      <parent link="${arm_id}_link7"/>
-      <child link="${arm_id}_link8"/>
-      <axis xyz="0 0 0"/>
-    </joint>
-  </xacro:macro>
+  <xacro:include filename="$(find franka_description)/robots/panda_arm.urdf.xacro"/>
+  <xacro:panda_arm />
   <xacro:include filename="$(find ros_objslampp_panda)/robots/suction/suction_gripper.xacro"/>
-  <xacro:panda_arm />
   <xacro:suction_gripper ns="panda" rpy="${pi} 0 ${-pi/4}" xyz="0 0 0.0065" connected_to="panda_link8"/>
 </robot>
