Commit message: ros_objslampp_panda -> morefusion_panda

File: ros/morefusion_panda/robots/moveit/panda.srdf.xacro (robot description, xacro)
@@ -5,5 +5,5 @@
 -->
 <robot xmlns:xacro="http://www.ros.org/wiki/xacro" name="panda">
-  <xacro:include filename="$(find ros_objslampp_panda)/robots/moveit/panda.xacro" />
+  <xacro:include filename="$(find morefusion_panda)/robots/moveit/panda.xacro" />
   <xacro:panda_arm />
 </robot>

File: ros/morefusion_panda/robots/panda.urdf.xacro (robot description, xacro)
@@ -6,17 +6,17 @@
   <!-- }} arm -->
   <!-- gripper {{ -->
-  <xacro:include filename="$(find ros_objslampp_panda)/robots/suction_gripper.xacro"/>
+  <xacro:include filename="$(find morefusion_panda)/robots/suction_gripper.xacro"/>
   <xacro:suction_gripper ns="panda" rpy="${pi} 0 ${-pi/4}" xyz="0 0 0.0065" connected_to="panda_link8"/>
   <!-- }} gripper -->
   <!-- scene {{ -->
-  <xacro:include filename="$(find ros_objslampp_panda)/robots/scene/table.xacro"/>
+  <xacro:include filename="$(find morefusion_panda)/robots/scene/table.xacro"/>
   <xacro:table ns="panda" rpy="0 0 0" xyz="0.68 0 0.0375" connected_to="panda_link0"/>
-  <xacro:include filename="$(find ros_objslampp_panda)/robots/scene/left_wall.xacro"/>
+  <xacro:include filename="$(find morefusion_panda)/robots/scene/left_wall.xacro"/>
   <xacro:left_wall ns="panda" rpy="${pi/2} 0 0" xyz="0.68 0.65 0.6" connected_to="panda_link0"/>
-  <xacro:include filename="$(find ros_objslampp_panda)/robots/scene/front_wall.xacro"/>
+  <xacro:include filename="$(find morefusion_panda)/robots/scene/front_wall.xacro"/>
   <xacro:front_wall ns="panda" rpy="0 ${pi/2} 0" xyz="1.33 0 0.6" connected_to="panda_link0"/>
-  <xacro:include filename="$(find ros_objslampp_panda)/robots/scene/target_box.xacro"/>
+  <xacro:include filename="$(find morefusion_panda)/robots/scene/target_box.xacro"/>
   <xacro:target_box ns="panda" rpy="0 0 0" xyz="0.6 -0.45 0.075" connected_to="panda_link0"/>
-  <xacro:include filename="$(find ros_objslampp_panda)/robots/scene/distractor_box.xacro"/>
+  <xacro:include filename="$(find morefusion_panda)/robots/scene/distractor_box.xacro"/>
   <xacro:distractor_box ns="panda" rpy="0 0 0" xyz="0.665 0.445 0.0775" connected_to="panda_link0"/>
   <!-- }} scene -->

File: ros/morefusion_panda/robots/suction_gripper.xacro (robot description, xacro)
@@ -18,5 +18,5 @@
       <visual>
         <geometry>
-          <mesh filename="package://ros_objslampp_panda/meshes/visual/suction_mount.stl"/>
+          <mesh filename="package://morefusion_panda/meshes/visual/suction_mount.stl"/>
         </geometry>
         <material name="black"/>
@@ -32,5 +32,5 @@
       <visual>
         <geometry>
-          <mesh filename="package://ros_objslampp_panda/meshes/visual/suction_cup.stl"/>
+          <mesh filename="package://morefusion_panda/meshes/visual/suction_cup.stl"/>
         </geometry>
         <material name="green"/>
